File: BluePillClone/BluePillClone.kicad_sch (KiCad schematic)
At the start: 28 parts, among them J1 USB_B_Micro, J2 Conn_01x04_Pin, J3 Conn_01x04_Pin, J4 Conn_01x04_Pin, SW1 SW_SPDT, U1 STM32F103C8Tx, U2 AMS1117-3.3, Y1 16MHz

Commit message: Final Commit.
Got Bored Not continuing further.

Routing needed to be done.
Parts:
- added H1, H2, H3, H4: MountingHole, MountingHole:MountingHole_2.2mm_M2, symbol Mechanical:MountingHole
Other:
- note added: "Mounting Holes"
